File: Ver_2/SWR_02.kicad_pcb (KiCad board)
At the start: 2 copper layers, 99.1 x 96.5 mm, 19 parts, among them J1 Conn_Coaxial, J2 Conn_Coaxial, J3 Conn_01, J4 Conn_01

Commit message: Add files via upload
Updated files copied to Git
Parts:
- removed FID1: Fiducial, Fiducial:Fiducial_0.75mm_Mask1.5mm
- added H3: MountingHole, MountingHole:MountingHole_2.5mm_Pad_TopBottom, F.Cu at (146.1, 111.8)
- D1, D2: value D -> BAT46; footprint Diode_SMD:D_1812_4532Metric_Pad1.30x3.40mm_HandSolder -> Diode_SMD:D_SOD-123
- J3, J4: footprint SWR_01:SolderWire-2sqmm_1 -> Connector_Wire:SolderWire-0.75sqmm_1x01_D1.25mm_OD2.3mm
- moved J2 38.1 mm to (146.1, 76.2)
- moved R4 21.6 mm to (143.5, 92.7)
- moved R3 21.6 mm to (137.2, 92.7)
- moved L1A2 18.3 mm to (121.9, 43.2)
- moved L2A1 18.2 mm to (88.9, 62.2)
- moved D2 13.7 mm to (137.2, 101.6), turned to 90 degrees
- moved C2 10.9 mm to (144.8, 102.9)
- moved J4 8.03 mm to (137.2, 109.2)
- moved L2A2 7.65 mm to (97.2, 86.4)
- moved H2 6.35 mm to (54.6, 111.8)
- moved J3 2.84 mm to (54.6, 58.4), turned to 0 degrees
- moved C1 2.54 mm to (54.6, 50.8)
- moved R2 1.27 mm to (57.1, 41.9)
Routing:
- net /Fwd: track 918.3 -> 729.4 mm
- net /Signal_Out: track 1001.1 -> 840.5 mm
- net GND: track 244.3 -> 253.8 mm
- net /Refl: track 134.5 -> 129.0 mm
- net /Refl_Out: track 16.6 -> 11.6 mm
- net /Fwd_Out: track 10.1 -> 11.5 mm
Other:
- board size 99.1 x 96.5 mm -> 99.1 x 90.2 mm
- net class Default: trace_width 0.25 -> 0.4
