File: Ver_2/SWR_02.sch (KiCad schematic (older format))
At the start: 18 parts, among them J1 Conn_Coaxial, J2 Conn_Coaxial, J3 Conn_01, J4 Conn_01

Commit message: Add files via upload
Updated files copied to Git
Parts:
- added H3: MountingHole, MountingHole:MountingHole_2.5mm_Pad_TopBottom, symbol Mechanical:MountingHole
- D1, D2: value D -> BAT46; footprint Diode_SMD:D_1812_4532Metric_Pad1.30x3.40mm_HandSolder -> Diode_SMD:D_SOD-123
- J3, J4: footprint SWR_01:SolderWire-2sqmm_1 -> Connector_Wire:SolderWire-0.75sqmm_1x01_D1.25mm_OD2.3mm
Connections:
- wire segments 42 -> 40
Other:
- moved on the sheet: C1, C2, D1, D2, J2, J3, J4, L1A1, L1A2, L2A1, L2A2, R3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
